File: ATXMega32_USB.sch (KiCad schematic (older format))
At the start: 34 parts, among them IC1 ATXMEGA32A4U, P1 CONN_20, P2 CONN_3X2, P3 CONN_20, P4 MICROUSB, X1 CRYSTAL

Commit message: Board mit BAS70BRW (schlechtes Layout)
Signed-off-by: TheTesla <stefan.helmert@gmx.net>
Parts:
- removed D3, D4, D5, D6: DIODESCH, symbol DIODESCH
- added D4: BAS70BRW, symbol BAS70BRW
- renumbered D7 to D3, D8 to D5
Connections:
- wire segments 256 -> 259

Commit message: Update der Bestellnummern, Bauteilwerte
Parts:
- C1, C12, C13, C3, C9: value CP1 -> 4u7; Digi-Key Part Number (none) -> 311-1371-2-ND
- C10, C11: value C -> 22p; Digi-Key Part Number (none) -> CL21C220JCANNND-ND
- C2, C4, C5, C6, C7, C8: value C -> 100n; Digi-Key Part Number (none) -> CL21F104ZAANNND-ND
- D4: Digi-Key Part Number (none) -> BAS70BRW-TPTR-ND
- L1: value INDUCTOR -> 100n; Digi-Key Part Number (none) -> CV201210-R10K-ND
- L2: value 100nH -> 100n; Digi-Key Part Number (none) -> CV201210-R10K-ND
- P4: Digi-Key Part Number (none) -> 609-4613-2-ND; Manufacturer Part Number (none) -> 10118192-0001LF
- R1: value R -> 10k; Digi-Key Part Number (none) -> RMCF0805JG10K0-ND
- R2, R3, R4: value R -> 330; Digi-Key Part Number (none) -> RMCF0805JG330R-ND
- R5: value R -> 680; Digi-Key Part Number (none) -> RMCF0805JG680R-ND
Changed lines of the file:
@@
-EESchema Schematic File Version 2  date 06.04.2013 03:03:50
+EESchema Schematic File Version 2  date 06.04.2013 18:32:48
 LIBS:atmel
 LIBS:libtest
@@
 F 0 "D4" H 9500 1850 40  0000 C CNN
 F 1 "BAS70BRW" H 9400 2050 40  0000 C CNN
+F 3 "http://www.mccsemi.com/up_pdf/BAS70TW_DW-04_DW-05_DW-06_BRW(SOT-363).PDF" H 9400 1950 60  0001 C CNN
+F 4 "BAS70BRW-TPTR-ND" H 9400 1950 60  0001 C CNN "Digi-Key Part Number"
 	2    9400 1950
 	0    -1   -1   0
@@
 P 9750 1600
 F 0 "R5" V 9830 1600 50  0000 C CNN
-F 1 "R" V 9750 1600 50  0000 C CNN
+F 1 "680" V 9750 1600 50  0000 C CNN
+F 3 "http://www.seielect.com/Catalog/SEI-RMCF_RMCP.pdf" H 9750 1600 60  0001 C CNN
+F 4 "RMCF0805JG680R-ND" V 9750 1600 60  0001 C CNN "Digi-Key Part Number"
 	1    9750 1600
 	-1   0    0    1
@@
 P 6100 1100
 F 0 "R4" V 6180 1100 50  0000 C CNN
-F 1 "R" V 6100 1100 50  0000 C CNN
+F 1 "330" V 6100 1100 50  0000 C CNN
+F 3 "http://www.seielect.com/Catalog/SEI-RMCF_RMCP.pdf" H 6100 1100 60  0001 C CNN
+F 4 "RMCF0805JG330R-ND" V 6100 1100 60  0001 C CNN "Digi-Key Part Number"
 	1    6100 1100
 	0    1    1    0
@@
 F 0 "P4" H 7850 1650 60  0000 C CNN
 F 1 "MICROUSB" H 8000 1550 60  0000 C CNN
+F 3 "http://portal.fciconnect.com/Comergent//fci/drawing/10118192.pdf" H 7950 1250 60  0001 C CNN
+F 4 "609-4613-2-ND" H 7950 1250 60  0001 C CNN "Digi-Key Part Number"
+F 5 "10118192-0001LF" H 7950 1250 60  0001 C CNN "Manufacturer Part Number"
 	1    7950 1250
 	0    1    1    0
@@
 P 7050 1700
 F 0 "R2" V 7130 1700 50  0000 C CNN
-F 1 "R" V 7050 1700 50  0000 C CNN
+F 1 "330" V 7050 1700 50  0000 C CNN
+F 3 "http://www.seielect.com/Catalog/SEI-RMCF_RMCP.pdf" H 7050 1700 60  0001 C CNN
+F 4 "RMCF0805JG330R-ND" V 7050 1700 60  0001 C CNN "Digi-Key Part Number"
 	1    7050 1700
 	-1   0    0    1
@@
 P 7350 1700
 F 0 "R3" V 7430 1700 50  0000 C CNN
-F 1 "R" V 7350 1700 50  0000 C CNN
+F 1 "330" V 7350 1700 50  0000 C CNN
+F 3 "http://www.seielect.com/Catalog/SEI-RMCF_RMCP.pdf" H 7350 1700 60  0001 C CNN
+F 4 "RMCF0805JG330R-ND" V 7350 1700 60  0001 C CNN "Digi-Key Part Number"
 	1    7350 1700
 	-1   0    0    1
@@
 P 6550 1950
 F 0 "C13" H 6600 2050 50  0000 L CNN
-F 1 "CP1" H 6600 1850 50  0000 L CNN
+F 1 "4u7" H 6600 1850 50  0000 L CNN
+F 3 "http://www.yageo.com/documents/recent/UPY-GPHC_Y5V_6.3V-to-50V_5.pdf" H 6550 1950 60  0001 C CNN
+F 4 "311-1371-2-ND" H 6550 1950 60  0001 C CNN "Digi-Key Part Number"
 	1    6550 1950
 	1    0    0    -1
@@
 P 4100 1700
 F 0 "C12" H 4150 1800 50  0000 L CNN
-F 1 "CP1" H 4150 1600 50  0000 L CNN
+F 1 "4u7" H 4150 1600 50  0000 L CNN
+F 3 "http://www.yageo.com/documents/recent/UPY-GPHC_Y5V_6.3V-to-50V_5.pdf" H 4100 1700 60  0001 C CNN
+F 4 "311-1371-2-ND" H 4100 1700 60  0001 C CNN "Digi-Key Part Number"
 	1    4100 1700
 	0    1    1    0
@@
 P 2550 900
 F 0 "L1" V 2500 900 40  0000 C CNN
-F 1 "INDUCTOR" V 2650 900 40  0000 C CNN
+F 1 "100n" V 2650 900 40  0000 C CNN
+F 3 "http://www.bourns.com/data/global/pdfs/CV201210.pdf" H 2550 900 60  0001 C CNN
+F 4 "CV201210-R10K-ND" H 2550 900 60  0001 C CNN "Digi-Key Part Number"
 	1    2550 900
 	0    -1   -1   0
@@
 P 3150 5600
 F 0 "C3" H 3200 5700 50  0000 L CNN
-F 1 "CP1" H 3200 5500 50  0000 L CNN
+F 1 "4u7" H 3200 5500 50  0000 L CNN
+F 3 "http://www.yageo.com/documents/recent/UPY-GPHC_Y5V_6.3V-to-50V_5.pdf" H 3150 5600 60  0001 C CNN
+F 4 "311-1371-2-ND" H 3150 5600 60  0001 C CNN "Digi-Key Part Number"
 	1    3150 5600
 	1    0    0    -1
@@
 P 2650 5600
 F 0 "C1" H 2700 5700 50  0000 L CNN
-F 1 "CP1" H 2700 5500 50  0000 L CNN
+F 1 "4u7" H 2700 5500 50  0000 L CNN
+F 3 "http://www.yageo.com/documents/recent/UPY-GPHC_Y5V_6.3V-to-50V_5.pdf" H 2650 5600 60  0001 C CNN
+F 4 "311-1371-2-ND" H 2650 5600 60  0001 C CNN "Digi-Key Part Number"
 	1    2650 5600
 	1    0    0    -1
@@
 P 2900 5600
 F 0 "C2" H 2950 5700 50  0000 L CNN
-F 1 "C" H 2950 5500 50  0000 L CNN
+F 1 "100n" H 2950 5500 50  0000 L CNN
+F 3 "http://www.samsungsem.com/servlet/DownloadServlet?dir=partnumber&num=&fileName=CL21F104ZAANNND.pdf" H 2900 5600 60  0001 C CNN
+F 4 "CL21F104ZAANNND-ND" H 2900 5600 60  0001 C CNN "Digi-Key Part Number"
 	1    2900 5600
 	1    0    0    -1
@@
 P 3400 5600
 F 0 "C4" H 3450 5700 50  0000 L CNN
-F 1 "C" H 3450 5500 50  0000 L CNN
+F 1 "100n" H 3450 5500 50  0000 L CNN
+F 3 "http://www.samsungsem.com/servlet/DownloadServlet?dir=partnumber&num=&fileName=CL21F104ZAANNND.pdf" H 3400 5600 60  0001 C CNN
+F 4 "CL21F104ZAANNND-ND" H 3400 5600 60  0001 C CNN "Digi-Key Part Number"
 	1    3400 5600
 	1    0    0    -1
@@
 P 7500 5600
 F 0 "C11" H 7550 5700 50  0000 L CNN
-F 1 "C" H 7550 5500 50  0000 L CNN
+F 1 "22p" H 7550 5500 50  0000 L CNN
+F 3 "http://www.samsungsem.com/servlet/DownloadServlet?dir=partnumber&num=&fileName=CL21C220JCANNND.pdf" H 7500 5600 60  0001 C CNN
+F 4 "CL21C220JCANNND-ND" H 7500 5600 60  0001 C CNN "Digi-Key Part Number"
 	1    7500 5600
 	1    0    0    -1
@@
 P 6650 5600
 F 0 "C10" H 6700 5700 50  0000 L CNN
-F 1 "C" H 6700 5500 50  0000 L CNN
+F 1 "22p" H 6700 5500 50  0000 L CNN
+F 3 "http://www.samsungsem.com/servlet/DownloadServlet?dir=partnumber&num=&fileName=CL21C220JCANNND.pdf" H 6650 5600 60  0001 C CNN
+F 4 "CL21C220JCANNND-ND" H 6650 5600 60  0001 C CNN "Digi-Key Part Number"
 	1    6650 5600
 	1    0    0    -1
@@
 P 6200 1950
 F 0 "C9" H 6250 2050 50  0000 L CNN
-F 1 "CP1" H 6250 1850 50  0000 L CNN
+F 1 "4u7" H 6250 1850 50  0000 L CNN
+F 3 "http://www.yageo.com/documents/recent/UPY-GPHC_Y5V_6.3V-to-50V_5.pdf" H 6200 1950 60  0001 C CNN
+F 4 "311-1371-2-ND" H 6200 1950 60  0001 C CNN "Digi-Key Part Number"
 	1    6200 1950
 	1    0    0    -1
@@
 P 4400 1400
 F 0 "L2" V 4350 1400 40  0000 C CNN
-F 1 "100nH" V 4500 1400 40  0000 C CNN
+F 1 "100n" V 4500 1400 40  0000 C CNN
+F 3 "http://www.bourns.com/data/global/pdfs/CV201210.pdf" H 4400 1400 60  0001 C CNN
+F 4 "CV201210-R10K-ND" H 4400 1400 60  0001 C CNN "Digi-Key Part Number"
 	1    4400 1400
 	1    0    0    -1
@@
 U 1 1 50BFC88B
 P 4100 2050
-F 0 "C5" H 4150 2150 50  0000 L CNN
-F 1 "C" H 4150 1950 50  0000 L CNN
+F 0 "C5" H 3950 1950 50  0000 L CNN
+F 1 "100n" H 3900 2150 50  0000 L CNN
+F 3 "http://www.samsungsem.com/servlet/DownloadServlet?dir=partnumber&num=&fileName=CL21F104ZAANNND.pdf" H 4100 2050 60  0001 C CNN
+F 4 "CL21F104ZAANNND-ND" H 4100 2050 60  0001 C CNN "Digi-Key Part Number"
 	1    4100 2050
 	0    -1   -1   0
@@
 P 5900 1950
 F 0 "C8" H 5950 2050 50  0000 L CNN
-F 1 "C" H 5950 1850 50  0000 L CNN
+F 1 "100n" H 5950 1850 50  0000 L CNN
+F 3 "http://www.samsungsem.com/servlet/DownloadServlet?dir=partnumber&num=&fileName=CL21F104ZAANNND.pdf" H 5900 1950 60  0001 C CNN
+F 4 "CL21F104ZAANNND-ND" H 5900 1950 60  0001 C CNN "Digi-Key Part Number"
 	1    5900 1950
 	1    0    0    -1
@@
 P 5600 1950
 F 0 "C7" H 5650 2050 50  0000 L CNN
-F 1 "C" H 5650 1850 50  0000 L CNN
+F 1 "100n" H 5650 1850 50  0000 L CNN
+F 3 "http://www.samsungsem.com/servlet/DownloadServlet?dir=partnumber&num=&fileName=CL21F104ZAANNND.pdf" H 5600 1950 60  0001 C CNN
+F 4 "CL21F104ZAANNND-ND" H 5600 1950 60  0001 C CNN "Digi-Key Part Number"
 	1    5600 1950
 	1    0    0    -1
@@
 P 5300 1950
 F 0 "C6" H 5350 2050 50  0000 L CNN
-F 1 "C" H 5350 1850 50  0000 L CNN
+F 1 "100n" H 5350 1850 50  0000 L CNN
+F 3 "http://www.samsungsem.com/servlet/DownloadServlet?dir=partnumber&num=&fileName=CL21F104ZAANNND.pdf" H 5300 1950 60  0001 C CNN
+F 4 "CL21F104ZAANNND-ND" H 5300 1950 60  0001 C CNN "Digi-Key Part Number"
 	1    5300 1950
 	1    0    0    -1
@@
 P 3500 2250
 F 0 "R1" V 3580 2250 50  0000 C CNN
-F 1 "R" V 3500 2250 50  0000 C CNN
+F 1 "10k" V 3500 2250 50  0000 C CNN
+F 3 "http://www.seielect.com/Catalog/SEI-RMCF_RMCP.pdf" H 3500 2250 60  0001 C CNN
+F 4 "RMCF0805JG10K0-ND" V 3500 2250 60  0001 C CNN "Digi-Key Part Number"
 	1    3500 2250
 	1    0    0    -1

Commit message: Z-Diode (USB ESD)
Signed-off-by: TheTesla <stefan.helmert@gmx.net>
Parts:
- added D6: 6V2, ~, symbol ZENER
- C10: value 22p -> 18p; Digi-Key Part Number CL21C220JCANNND-ND -> CL21C180JBANNND-ND; Manufacturer Part Number (none) -> CL21C180JBANNND
- C11: value 22p -> 18p; Digi-Key Part Number CL21C220JCANNND-ND -> CL21C180JBANNND-ND
- D1: Color (none) -> green; Digi-Key Part Number (none) -> 160-1426-2-ND; Manufacturer Part Number (none) -> LTST-C171KGKT
- D2: Color (none) -> red; Digi-Key Part Number (none) -> 160-1415-2-ND; Manufacturer Part Number (none) -> LTST-C170KRKT
- D3: Color (none) -> yellow; Digi-Key Part Number (none) -> 160-1416-2-ND; Manufacturer Part Number (none) -> 160-1416-2-ND
- D5: Color (none) -> blue; Digi-Key Part Number (none) -> 160-1645-2-ND; Manufacturer Part Number (none) -> LTST-C171TBKT
- IC1: Alternative (none) -> ATXMEGA128A4U-AU-ND; Digi-Key Part Number (none) -> ATXMEGA32A4U-AURTR-ND
- P1, P3: CSD-Electronics Part Number (none) -> 15435; Notes (none) -> 1/2 of Part
- P2: CSD-Electronics Part Number (none) -> 15485; Notes (none) -> 3/40 of Part
- X1: value CRYSTAL -> 4 MHz; Digi-Key Part Number (none) -> 535-9057-ND; Manufacturer Part Number (none) -> ABL-4.000MHZ-B2
Connections:
- net GND: now also D6.1 (A)
- net at D4.4 (cathode), D4.5 (cathode), P3.1 (P1)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: now also D6.2 (K)
- no-connect marks 2 -> 3
Other:
- note added: "ATXMega USB Breakout Board"

Commit message: Update BOM, Rename-Script
Signed-off-by: TheTesla <stefan.helmert@gmx.net>
Parts:
- C1, C10, C11, C12, C13, C3, C9, D3, D5, L1, L2, R1, R2, R3, R4, R5: footprint (none) -> SM0805
- C2, C4, C5, C6, C7, C8: footprint (none) -> SM0603_Capa
- D1, D2: footprint (none) -> LED-0805
- D4: footprint (none) -> SOT363
- D4: footprint (none) -> SOT363; Digi-Key Part Number (none) -> BAS70BRW-TPTR-ND
- D6: footprint ~ -> SOD323
- P1, P3: footprint (none) -> PIN_ARRAY_20X1; CSD-Electronics Part Number 15435 -> CSD-Electronics: 15435
- P2: footprint (none) -> pin_array_3x2; CSD-Electronics Part Number 15485 -> CSD-Electronics: 15485; Notes 3/40 of Part -> 3/40 of Part
- P4: footprint (none) -> ZX62-B-5PA
- X1: footprint (none) -> HC-49V

Commit message: Seeed OPL SKU ergänzt; csv mit neuem eigenem xsl-Plugin
Signed-off-by: TheTesla <stefan.helmert@gmx.net>
Parts:
- C1, C12, C13, C3, C9: value 4u7 -> 10u; Seeed OPL SKU (none) -> 010008001
- C2, C4, C5, C6, C7, C8: Seeed OPL SKU (none) -> 010002001
- D1: Seeed OPL SKU (none) -> 033003001
- D2: Seeed OPL SKU (none) -> 033004001
- P1, P3: CSD-Electronics Part Number CSD-Electronics: 15435 -> 15435
- P2: CSD-Electronics Part Number CSD-Electronics: 15485 -> 15485
- R1: Seeed OPL SKU (none) -> 002004001
- R2, R3, R4: value 330 -> 1k; Seeed OPL SKU (none) -> 002011001
- R5: value 680 -> 1k5; Seeed OPL SKU (none) -> 002022001
Changed lines of the file:
@@
-EESchema Schematic File Version 2  date 07.04.2013 03:00:35
+EESchema Schematic File Version 2  date 15.04.2013 23:52:48
 LIBS:atmel
 LIBS:libtest
@@
 Sheet 1 1
 Title ""
-Date "7 apr 2013"
+Date "15 apr 2013"
 Rev ""
 Comp ""
@@
 F 1 "BAS70BRW" H 9100 2050 40  0000 C CNN
 F 2 "SOT363" H 9100 1950 60  0001 C CNN
-F 3 "~" H 9100 1950 60  0001 C CNN
+F 3 "http://www.mccsemi.com/up_pdf/BAS70TW_DW-04_DW-05_DW-06_BRW(SOT-363).PDF" H 9100 1950 60  0001 C CNN
 F 4 "BAS70BRW-TPTR-ND" H 9100 1950 60  0001 C CNN "Digi-Key Part Number"
 F 5 "~" H 9100 1950 60  0001 C CNN "Manufacturer Part Number"
@@
 F 1 "BAS70BRW" H 9400 2050 40  0000 C CNN
 F 2 "SOT363" H 9400 1950 60  0001 C CNN
-F 3 "~" H 9400 1950 60  0001 C CNN
+F 3 "http://www.mccsemi.com/up_pdf/BAS70TW_DW-04_DW-05_DW-06_BRW(SOT-363).PDF" H 9400 1950 60  0001 C CNN
 F 4 "BAS70BRW-TPTR-ND" H 9400 1950 60  0001 C CNN "Digi-Key Part Number"
 F 5 "~" H 9400 1950 60  0001 C CNN "Manufacturer Part Number"
@@
 P 9750 1600
 F 0 "R5" V 9830 1600 50  0000 C CNN
-F 1 "680" V 9750 1600 50  0000 C CNN
+F 1 "1k5" V 9750 1600 50  0000 C CNN
 F 2 "SM0805" H 9750 1600 60  0001 C CNN
 F 3 "http://www.seielect.com/Catalog/SEI-RMCF_RMCP.pdf" H 9750 1600 60  0001 C CNN
 F 4 "RMCF0805JG680R-ND" V 9750 1600 60  0001 C CNN "Digi-Key Part Number"
+F 5 "002022001" H 9750 1600 60  0001 C CNN "Seeed OPL SKU"
 	1    9750 1600
 	-1   0    0    1
@@
 P 6100 1100
 F 0 "R4" V 6180 1100 50  0000 C CNN
-F 1 "330" V 6100 1100 50  0000 C CNN
+F 1 "1k" V 6100 1100 50  0000 C CNN
 F 2 "SM0805" H 6100 1100 60  0001 C CNN
 F 3 "http://www.seielect.com/Catalog/SEI-RMCF_RMCP.pdf" H 6100 1100 60  0001 C CNN
 F 4 "RMCF0805JG330R-ND" V 6100 1100 60  0001 C CNN "Digi-Key Part Number"
+F 5 "002011001" H 6100 1100 60  0001 C CNN "Seeed OPL SKU"
 	1    6100 1100
 	0    1    1    0
@@
 P 7050 1700
 F 0 "R2" V 7130 1700 50  0000 C CNN
-F 1 "330" V 7050 1700 50  0000 C CNN
+F 1 "1k" V 7050 1700 50  0000 C CNN
 F 2 "SM0805" H 7050 1700 60  0001 C CNN
 F 3 "http://www.seielect.com/Catalog/SEI-RMCF_RMCP.pdf" H 7050 1700 60  0001 C CNN
 F 4 "RMCF0805JG330R-ND" V 7050 1700 60  0001 C CNN "Digi-Key Part Number"
+F 5 "002011001" H 7050 1700 60  0001 C CNN "Seeed OPL SKU"
 	1    7050 1700
 	-1   0    0    1
@@
 P 7350 1700
 F 0 "R3" V 7430 1700 50  0000 C CNN
-F 1 "330" V 7350 1700 50  0000 C CNN
+F 1 "1k" V 7350 1700 50  0000 C CNN
 F 2 "SM0805" H 7350 1700 60  0001 C CNN
 F 3 "http://www.seielect.com/Catalog/SEI-RMCF_RMCP.pdf" H 7350 1700 60  0001 C CNN
 F 4 "RMCF0805JG330R-ND" V 7350 1700 60  0001 C CNN "Digi-Key Part Number"
+F 5 "002011001" H 7350 1700 60  0001 C CNN "Seeed OPL SKU"
 	1    7350 1700
 	-1   0    0    1
@@
 F 4 "160-1415-2-ND" H 7350 2200 60  0001 C CNN "Digi-Key Part Number"
 F 5 "LTST-C170KRKT" H 7350 2200 60  0001 C CNN "Manufacturer Part Number"
-F 6 "red" H 7350 2200 60  0001 C CNN "Color"
+F 6 "033004001" H 7350 2200 60  0001 C CNN "Seeed OPL SKU"
+F 7 "red" H 7350 2200 60  0001 C CNN "Color"
 	1    7350 2200
 	0    1    1    0
@@
 F 4 "160-1426-2-ND" H 7050 2200 60  0001 C CNN "Digi-Key Part Number"
 F 5 "LTST-C171KGKT" H 7050 2200 60  0001 C CNN "Manufacturer Part Number"
-F 6 "green" H 7050 2200 60  0001 C CNN "Color"
+F 6 "033003001" H 7050 2200 60  0001 C CNN "Seeed OPL SKU"
+F 7 "green" H 7050 2200 60  0001 C CNN "Color"
 	1    7050 2200
 	0    1    1    0
@@
 P 6550 1950
 F 0 "C13" H 6600 2050 50  0000 L CNN
-F 1 "4u7" H 6600 1850 50  0000 L CNN
+F 1 "10u" H 6600 1850 50  0000 L CNN
 F 2 "SM0805" H 6550 1950 60  0001 C CNN
 F 3 "http://www.yageo.com/documents/recent/UPY-GPHC_Y5V_6.3V-to-50V_5.pdf" H 6550 1950 60  0001 C CNN
 F 4 "311-1371-2-ND" H 6550 1950 60  0001 C CNN "Digi-Key Part Number"
+F 5 "010008001" H 6550 1950 60  0001 C CNN "Seeed OPL SKU"
 	1    6550 1950
 	1    0    0    -1
@@
 P 4100 1700
 F 0 "C12" H 4150 1800 50  0000 L CNN
-F 1 "4u7" H 4150 1600 50  0000 L CNN
+F 1 "10u" H 4150 1600 50  0000 L CNN
 F 2 "SM0805" H 4100 1700 60  0001 C CNN
 F 3 "http://www.yageo.com/documents/recent/UPY-GPHC_Y5V_6.3V-to-50V_5.pdf" H 4100 1700 60  0001 C CNN
 F 4 "311-1371-2-ND" H 4100 1700 60  0001 C CNN "Digi-Key Part Number"
+F 5 "010008001" H 4100 1700 60  0001 C CNN "Seeed OPL SKU"
 	1    4100 1700
 	0    1    1    0
@@
 F 5 "~" H 9000 4400 60  0001 C CNN "Manufacturer Part Number"
 F 6 "1/2 of Part" H 9000 4400 60  0001 C CNN "Notes"
-F 7 "CSD-Electronics: 15435" V 9000 4400 60  0001 C CNN "CSD-Electronics Part Number"
+F 7 "15435" V 9000 4400 60  0001 C CNN "CSD-Electronics Part Number"
 	1    9000 4400
 	1    0    0    -1
@@
 F 5 "~" H 1050 5000 60  0001 C CNN "Manufacturer Part Number"
 F 6 "1/2 of Part" H 1050 5000 60  0001 C CNN "Notes"
-F 7 "CSD-Electronics: 15435" V 1050 5000 60  0001 C CNN "CSD-Electronics Part Number"
+F 7 "15435" V 1050 5000 60  0001 C CNN "CSD-Electronics Part Number"
 	1    1050 5000
 	-1   0    0    -1
@@
 P 3150 5600
 F 0 "C3" H 3200 5700 50  0000 L CNN
-F 1 "4u7" H 3200 5500 50  0000 L CNN
+F 1 "10u" H 3200 5500 50  0000 L CNN
 F 2 "SM0805" H 3150 5600 60  0001 C CNN
 F 3 "http://www.yageo.com/documents/recent/UPY-GPHC_Y5V_6.3V-to-50V_5.pdf" H 3150 5600 60  0001 C CNN
 F 4 "311-1371-2-ND" H 3150 5600 60  0001 C CNN "Digi-Key Part Number"
+F 5 "010008001" H 3150 5600 60  0001 C CNN "Seeed OPL SKU"
 	1    3150 5600
 	1    0    0    -1
@@
 P 2650 5600
 F 0 "C1" H 2700 5700 50  0000 L CNN
-F 1 "4u7" H 2700 5500 50  0000 L CNN
+F 1 "10u" H 2700 5500 50  0000 L CNN
 F 2 "SM0805" H 2650 5600 60  0001 C CNN
 F 3 "http://www.yageo.com/documents/recent/UPY-GPHC_Y5V_6.3V-to-50V_5.pdf" H 2650 5600 60  0001 C CNN
 F 4 "311-1371-2-ND" H 2650 5600 60  0001 C CNN "Digi-Key Part Number"
+F 5 "010008001" H 2650 5600 60  0001 C CNN "Seeed OPL SKU"
 	1    2650 5600
 	1    0    0    -1
@@
 F 3 "http://www.samsungsem.com/servlet/DownloadServlet?dir=partnumber&num=&fileName=CL21F104ZAANNND.pdf" H 2900 5600 60  0001 C CNN
 F 4 "CL21F104ZAANNND-ND" H 2900 5600 60  0001 C CNN "Digi-Key Part Number"
+F 5 "010002001" H 2900 5600 60  0001 C CNN "Seeed OPL SKU"
 	1    2900 5600
 	1    0    0    -1
@@
 F 3 "http://www.samsungsem.com/servlet/DownloadServlet?dir=partnumber&num=&fileName=CL21F104ZAANNND.pdf" H 3400 5600 60  0001 C CNN
 F 4 "CL21F104ZAANNND-ND" H 3400 5600 60  0001 C CNN "Digi-Key Part Number"
+F 5 "010002001" H 3400 5600 60  0001 C CNN "Seeed OPL SKU"
 	1    3400 5600
 	1    0    0    -1
@@
 P 6200 1950
 F 0 "C9" H 6250 2050 50  0000 L CNN
-F 1 "4u7" H 6250 1850 50  0000 L CNN
+F 1 "10u" H 6250 1850 50  0000 L CNN
 F 2 "SM0805" H 6200 1950 60  0001 C CNN
 F 3 "http://www.yageo.com/documents/recent/UPY-GPHC_Y5V_6.3V-to-50V_5.pdf" H 6200 1950 60  0001 C CNN
 F 4 "311-1371-2-ND" H 6200 1950 60  0001 C CNN "Digi-Key Part Number"
+F 5 "010008001" H 6200 1950 60  0001 C CNN "Seeed OPL SKU"
 	1    6200 1950
 	1    0    0    -1
@@
 F 3 "http://www.samsungsem.com/servlet/DownloadServlet?dir=partnumber&num=&fileName=CL21F104ZAANNND.pdf" H 4100 2050 60  0001 C CNN
 F 4 "CL21F104ZAANNND-ND" H 4100 2050 60  0001 C CNN "Digi-Key Part Number"
+F 5 "010002001" H 4100 2050 60  0001 C CNN "Seeed OPL SKU"
 	1    4100 2050
 	0    -1   -1   0
@@
 F 3 "http://www.samsungsem.com/servlet/DownloadServlet?dir=partnumber&num=&fileName=CL21F104ZAANNND.pdf" H 5900 1950 60  0001 C CNN
 F 4 "CL21F104ZAANNND-ND" H 5900 1950 60  0001 C CNN "Digi-Key Part Number"
+F 5 "010002001" H 5900 1950 60  0001 C CNN "Seeed OPL SKU"
 	1    5900 1950
 	1    0    0    -1
@@
 F 3 "http://www.samsungsem.com/servlet/DownloadServlet?dir=partnumber&num=&fileName=CL21F104ZAANNND.pdf" H 5600 1950 60  0001 C CNN
 F 4 "CL21F104ZAANNND-ND" H 5600 1950 60  0001 C CNN "Digi-Key Part Number"
+F 5 "010002001" H 5600 1950 60  0001 C CNN "Seeed OPL SKU"
 	1    5600 1950
 	1    0    0    -1
@@
 F 3 "http://www.samsungsem.com/servlet/DownloadServlet?dir=partnumber&num=&fileName=CL21F104ZAANNND.pdf" H 5300 1950 60  0001 C CNN
 F 4 "CL21F104ZAANNND-ND" H 5300 1950 60  0001 C CNN "Digi-Key Part Number"
+F 5 "010002001" H 5300 1950 60  0001 C CNN "Seeed OPL SKU"
 	1    5300 1950
 	1    0    0    -1
@@
 F 3 "http://www.seielect.com/Catalog/SEI-RMCF_RMCP.pdf" H 3500 2250 60  0001 C CNN
 F 4 "RMCF0805JG10K0-ND" V 3500 2250 60  0001 C CNN "Digi-Key Part Number"
+F 5 "002004001" H 3500 2250 60  0001 C CNN "Seeed OPL SKU"
 	1    3500 2250
 	1    0    0    -1
@@
 F 5 "~" H 2850 2650 60  0001 C CNN "Manufacturer Part Number"
 F 6 "3/40 of Part " H 2850 2650 60  0001 C CNN "Notes"
-F 7 "CSD-Electronics: 15485" H 2850 2650 60  0001 C CNN "CSD-Electronics Part Number"
+F 7 "15485" H 2850 2650 60  0001 C CNN "CSD-Electronics Part Number"
 	1    2850 2650
 	-1   0    0    1

Commit message: removed space from one Digi-Key Part Number
Signed-off-by: TheTesla <stefan.helmert@gmx.net>
Parts:
- D6: Digi-Key Part Number SZMM3Z6V2T1G-ND -> SZMM3Z6V2T1G-ND
- P2: Seeed OPL SKU (none) -> 346018001
Changed lines of the file:
@@
-EESchema Schematic File Version 2  date 15.04.2013 23:52:48
+EESchema Schematic File Version 2  date 20.04.2013 01:52:58
 LIBS:atmel
 LIBS:libtest
@@
 Sheet 1 1
 Title ""
-Date "15 apr 2013"
+Date "19 apr 2013"
 Rev ""
 Comp ""
@@
 F 5 "~" H 2850 2650 60  0001 C CNN "Manufacturer Part Number"
 F 6 "3/40 of Part " H 2850 2650 60  0001 C CNN "Notes"
-F 7 "15485" H 2850 2650 60  0001 C CNN "CSD-Electronics Part Number"
+F 7 "346018001" H 2850 2650 60  0001 C CNN "Seeed OPL SKU"
+F 8 "15485" H 2850 2650 60  0001 C CNN "CSD-Electronics Part Number"
 	1    2850 2650
 	-1   0    0    1
@@
 F 2 "SOD323" H 10100 1850 60  0001 C CNN
 F 3 "http://www.onsemi.com/pub_link/Collateral/MM3Z2V4T1-D.PDF" H 10100 2150 60  0001 C CNN
-F 4 "SZMM3Z6V2T1G-ND	" H 10100 2150 60  0001 C CNN "Digi-Key Part Number"
+F 4 "SZMM3Z6V2T1G-ND" H 10100 2150 60  0001 C CNN "Digi-Key Part Number"
 	1    10100 2150
 	0    -1   -1   0

Commit message: updated parts - BOM
Signed-off-by: TheTesla <stefan.helmert@gmx.net>
Parts:
- C1, C12, C13, C3, C9: Digi-Key Part Number 311-1371-2-ND -> 445-1372-1-ND; Manufacturer Part Number (none) -> C2012Y5V0J106Z
- C10: Digi-Key Part Number CL21C180JBANNND-ND -> 1276-1107-1-ND; Manufacturer Part Number CL21C180JBANNND -> CL21C180JBANNNC
- C11: Digi-Key Part Number CL21C180JBANNND-ND -> 1276-1107-1-ND; Manufacturer Part Number (none) -> CL21C180JBANNNC
- C2, C4, C5, C6, C7, C8: Digi-Key Part Number CL21F104ZAANNND-ND -> 445-7534-1-ND; Manufacturer Part Number (none) -> C2012X7R1H104K085AA
- D4: Digi-Key Part Number BAS70BRW-TPTR-ND -> BAS70BRW-TPCT-ND
- D6: Digi-Key Part Number SZMM3Z6V2T1G-ND -> MM3Z6V2ST1GOSCT-ND; Manufacturer Part Number (none) -> MM3Z6V2ST1G
- IC1: Digi-Key Part Number ATXMEGA32A4U-AURTR-ND -> ATXMEGA32A4U-AU-ND
- L1, L2: Digi-Key Part Number CV201210-R10K-ND -> 535-11645-1-ND; Manufacturer Part Number (none) -> AIML-0805-R10K-T
- R2, R3, R4: Digi-Key Part Number RMCF0805JG330R-ND -> RMCF0805JT1K00CT-ND; Manufacturer Part Number (none) -> RMCF0805JT1K00
- R5: Digi-Key Part Number RMCF0805JG680R-ND -> RMCF0805JT1K50CT-ND; Manufacturer Part Number (none) -> RMCF0805JT1K50
- X1: Digi-Key Part Number 535-9057-ND -> CTX896-ND; Manufacturer Part Number ABL-4.000MHZ-B2 -> ATS040B
