File: ATXMega32_USB.sch (KiCad schematic (older format))
At the start: 32 parts, among them IC1 ATXMEGA32A4U, P1 CONN_20, P2 CONN_3X2, P3 CONN_20, P4 MICROUSB, X1 4 MHz

Commit message: components changed: cheaper leds, minimum quantity 1, no obsolete parts
Signed-off-by: TheTesla <stefan.helmert@gmx.net>
Parts:
- C1, C12, C13, C3, C9: Digi-Key Part Number 445-1372-1-ND -> 311-1355-1-ND; Manufacturer Part Number C2012Y5V0J106Z -> CC0805ZKY5V6BB106
- D1: Digi-Key Part Number 160-1426-2-ND -> 475-1410-1-ND; Manufacturer Part Number LTST-C171KGKT -> LG R971-KN-1
- D2: Digi-Key Part Number 160-1415-2-ND -> 475-1278-1-ND; Manufacturer Part Number LTST-C170KRKT -> LS R976-NR-1
- D3: Digi-Key Part Number 160-1416-2-ND -> 475-2560-1-ND; Manufacturer Part Number 160-1416-2-ND -> LY R976-PS-36
- D5: Digi-Key Part Number 160-1645-2-ND -> 160-1579-1-ND; Manufacturer Part Number LTST-C171TBKT -> LTST-C170TBKT
Changed lines of the file:
@@
-EESchema Schematic File Version 2  date 14.05.2013 16:40:03
+EESchema Schematic File Version 2  date 19.05.2013 04:39:10
 LIBS:atmel
 LIBS:libtest
@@
 Sheet 1 1
 Title ""
-Date "14 may 2013"
+Date "19 may 2013"
 Rev ""
 Comp ""
@@
 F 1 "LED" H 6550 1250 50  0000 C CNN
 F 2 "SM0805" H 6550 1350 60  0001 C CNN
-F 3 "http://optoelectronics.liteon.com/en-us/api/DwonloadFileHandler.ashx?txtSpecNo=DS-22-99-0188&txtPartNo=LTST-C170KSKT" H 6550 1350 60  0001 C CNN
-F 4 "160-1416-2-ND" H 6550 1350 60  0001 C CNN "Digi-Key Part Number"
-F 5 "160-1416-2-ND" H 6550 1350 60  0001 C CNN "Manufacturer Part Number"
+F 3 "http://catalog.osram-os.com/jsp/download.jsp?name=LO_LS_LY_R976.pdf&url=/media/_en/Graphics/00042116_0.pdf" H 6550 1350 60  0001 C CNN
+F 4 "475-2560-1-ND" H 6550 1350 60  0001 C CNN "Digi-Key Part Number"
+F 5 "LY R976-PS-36" H 6550 1350 60  0001 C CNN "Manufacturer Part Number"
 F 6 "yellow" H 6550 1350 60  0001 C CNN "Color"
 	1    6550 1350
@@
 F 1 "LED" H 9750 2050 50  0000 C CNN
 F 2 "SM0805" H 9750 2150 60  0001 C CNN
-F 3 "http://media.digikey.com/pdf/Data%20Sheets/Lite-On%20PDFs/LTST-C171TBKT.pdf" H 9750 2150 60  0001 C CNN
-F 4 "160-1645-2-ND" H 9750 2150 60  0001 C CNN "Digi-Key Part Number"
-F 5 "LTST-C171TBKT" H 9750 2150 60  0001 C CNN "Manufacturer Part Number"
+F 3 "http://optoelectronics.liteon.com/en-us/api/DwonloadFileHandler.ashx?txtSpecNo=DS-22-99-0226&txtPartNo=LTST-C170TBKT" H 9750 2150 60  0001 C CNN
+F 4 "160-1579-1-ND" H 9750 2150 60  0001 C CNN "Digi-Key Part Number"
+F 5 "LTST-C170TBKT" H 9750 2150 60  0001 C CNN "Manufacturer Part Number"
 F 6 "blue" H 9750 2150 60  0001 C CNN "Color"
 	1    9750 2150
@@
 F 1 "LED" H 7350 2100 50  0000 C CNN
 F 2 "LED-0805" H 7350 2200 60  0001 C CNN
-F 3 "http://optoelectronics.liteon.com/en-us/api/DwonloadFileHandler.ashx?txtSpecNo=DS-22-99-0150&txtPartNo=LTST-C170KRKT" H 7350 2200 60  0001 C CNN
-F 4 "160-1415-2-ND" H 7350 2200 60  0001 C CNN "Digi-Key Part Number"
-F 5 "LTST-C170KRKT" H 7350 2200 60  0001 C CNN "Manufacturer Part Number"
+F 3 "http://catalog.osram-os.com/jsp/download.jsp?name=LO_LS_LY_R976.pdf&url=/media/_en/Graphics/00042116_0.pdf" H 7350 2200 60  0001 C CNN
+F 4 "475-1278-1-ND" H 7350 2200 60  0001 C CNN "Digi-Key Part Number"
+F 5 "LS R976-NR-1" H 7350 2200 60  0001 C CNN "Manufacturer Part Number"
 F 6 "033004001" H 7350 2200 60  0001 C CNN "Seeed OPL SKU"
 F 7 "red" H 7350 2200 60  0001 C CNN "Color"
@@
 F 1 "LED" H 7050 2100 50  0000 C CNN
 F 2 "LED-0805" H 7050 2200 60  0001 C CNN
-F 3 "http://optoelectronics.liteon.com/en-us/api/DwonloadFileHandler.ashx?txtSpecNo=DS22-2000-118&txtPartNo=LTST-C171KGKT" H 7050 2200 60  0001 C CNN
-F 4 "160-1426-2-ND" H 7050 2200 60  0001 C CNN "Digi-Key Part Number"
-F 5 "LTST-C171KGKT" H 7050 2200 60  0001 C CNN "Manufacturer Part Number"
+F 3 "http://catalog.osram-os.com/catalogue/catalogue.do;jsessionid=B38D4035738FAE714C474120326E9384?act=downloadFile&favOid=02000002000009ee000100b6" H 7050 2200 60  0001 C CNN
+F 4 "475-1410-1-ND" H 7050 2200 60  0001 C CNN "Digi-Key Part Number"
+F 5 "LG R971-KN-1" H 7050 2200 60  0001 C CNN "Manufacturer Part Number"
 F 6 "033003001" H 7050 2200 60  0001 C CNN "Seeed OPL SKU"
 F 7 "green" H 7050 2200 60  0001 C CNN "Color"
@@
 F 1 "10u" H 6600 1850 50  0000 L CNN
 F 2 "SM0805" H 6550 1950 60  0001 C CNN
-F 3 "http://media.digikey.com/pdf/Data%20Sheets/TDK%20PDFs/C_Series_GeneralAppl_Spec_rev_0.3_201012.pdf" H 6550 1950 60  0001 C CNN
-F 4 "445-1372-1-ND" H 6550 1950 60  0001 C CNN "Digi-Key Part Number"
-F 5 "C2012Y5V0J106Z" H 6550 1950 60  0001 C CNN "Manufacturer Part Number"
+F 3 "http://www.yageo.com/documents/recent/UPY-GPHC_Y5V_6.3V-to-50V_5.pdf" H 6550 1950 60  0001 C CNN
+F 4 "311-1355-1-ND" H 6550 1950 60  0001 C CNN "Digi-Key Part Number"
+F 5 "CC0805ZKY5V6BB106" H 6550 1950 60  0001 C CNN "Manufacturer Part Number"
 F 6 "010008001" H 6550 1950 60  0001 C CNN "Seeed OPL SKU"
 	1    6550 1950
@@
 F 1 "10u" H 4150 1600 50  0000 L CNN
 F 2 "SM0805" H 4100 1700 60  0001 C CNN
-F 3 "http://media.digikey.com/pdf/Data%20Sheets/TDK%20PDFs/C_Series_GeneralAppl_Spec_rev_0.3_201012.pdf" H 4100 1700 60  0001 C CNN
-F 4 "445-1372-1-ND" H 4100 1700 60  0001 C CNN "Digi-Key Part Number"
-F 5 "C2012Y5V0J106Z" H 4100 1700 60  0001 C CNN "Manufacturer Part Number"
+F 3 "http://www.yageo.com/documents/recent/UPY-GPHC_Y5V_6.3V-to-50V_5.pdf" H 4100 1700 60  0001 C CNN
+F 4 "311-1355-1-ND" H 4100 1700 60  0001 C CNN "Digi-Key Part Number"
+F 5 "CC0805ZKY5V6BB106" H 4100 1700 60  0001 C CNN "Manufacturer Part Number"
 F 6 "010008001" H 4100 1700 60  0001 C CNN "Seeed OPL SKU"
 	1    4100 1700
@@
 F 1 "10u" H 3200 5500 50  0000 L CNN
 F 2 "SM0805" H 3150 5600 60  0001 C CNN
-F 3 "http://media.digikey.com/pdf/Data%20Sheets/TDK%20PDFs/C_Series_GeneralAppl_Spec_rev_0.3_201012.pdf" H 3150 5600 60  0001 C CNN
-F 4 "445-1372-1-ND" H 3150 5600 60  0001 C CNN "Digi-Key Part Number"
-F 5 "C2012Y5V0J106Z" H 3150 5600 60  0001 C CNN "Manufacturer Part Number"
+F 3 "http://www.yageo.com/documents/recent/UPY-GPHC_Y5V_6.3V-to-50V_5.pdf" H 3150 5600 60  0001 C CNN
+F 4 "311-1355-1-ND" H 3150 5600 60  0001 C CNN "Digi-Key Part Number"
+F 5 "CC0805ZKY5V6BB106" H 3150 5600 60  0001 C CNN "Manufacturer Part Number"
 F 6 "010008001" H 3150 5600 60  0001 C CNN "Seeed OPL SKU"
 	1    3150 5600
@@
 F 1 "10u" H 2700 5500 50  0000 L CNN
 F 2 "SM0805" H 2650 5600 60  0001 C CNN
-F 3 "http://media.digikey.com/pdf/Data%20Sheets/TDK%20PDFs/C_Series_GeneralAppl_Spec_rev_0.3_201012.pdf" H 2650 5600 60  0001 C CNN
-F 4 "445-1372-1-ND" H 2650 5600 60  0001 C CNN "Digi-Key Part Number"
-F 5 "C2012Y5V0J106Z" H 2650 5600 60  0001 C CNN "Manufacturer Part Number"
+F 3 "http://www.yageo.com/documents/recent/UPY-GPHC_Y5V_6.3V-to-50V_5.pdf" H 2650 5600 60  0001 C CNN
+F 4 "311-1355-1-ND" H 2650 5600 60  0001 C CNN "Digi-Key Part Number"
+F 5 "CC0805ZKY5V6BB106" H 2650 5600 60  0001 C CNN "Manufacturer Part Number"
 F 6 "010008001" H 2650 5600 60  0001 C CNN "Seeed OPL SKU"
 	1    2650 5600
@@
 F 1 "10u" H 6250 1850 50  0000 L CNN
 F 2 "SM0805" H 6200 1950 60  0001 C CNN
-F 3 "http://media.digikey.com/pdf/Data%20Sheets/TDK%20PDFs/C_Series_GeneralAppl_Spec_rev_0.3_201012.pdf" H 6200 1950 60  0001 C CNN
-F 4 "445-1372-1-ND" H 6200 1950 60  0001 C CNN "Digi-Key Part Number"
-F 5 "C2012Y5V0J106Z" H 6200 1950 60  0001 C CNN "Manufacturer Part Number"
+F 3 "http://www.yageo.com/documents/recent/UPY-GPHC_Y5V_6.3V-to-50V_5.pdf" H 6200 1950 60  0001 C CNN
+F 4 "311-1355-1-ND" H 6200 1950 60  0001 C CNN "Digi-Key Part Number"
+F 5 "CC0805ZKY5V6BB106" H 6200 1950 60  0001 C CNN "Manufacturer Part Number"
 F 6 "010008001" H 6200 1950 60  0001 C CNN "Seeed OPL SKU"
 	1    6200 1950
