File: ATXMega128_USB.sch (KiCad schematic (older format))
At the start: 32 parts, among them IC1 ATXMEGA32A4U, P1 CONN_20, P2 CONN_3X2, P3 CONN_20, P4 MICROUSB, X1 4 MHz

Commit message: board and schematic updated to atxmega128a4u
Parts:
- removed IC1: ATXMEGA32A4U, TQFP44, symbol ATXMEGA32A4U
- added IC?: ATXMEGA128A4U, TQFP44, symbol ATXMEGA128A4U
Changed lines of the file:
@@
-EESchema Schematic File Version 2  date 01.09.2013 12:46:57
+EESchema Schematic File Version 2  date 01.09.2013 16:25:21
 LIBS:atmel
 LIBS:libtest
@@
 Sheet 1 1
 Title ""
-Date "17 jul 2013"
+Date "1 sep 2013"
 Rev ""
 Comp ""
@@
 F 3 "" H 7700 2450 60  0001 C CNN
 	1    7700 2450
-	1    0    0    -1
-$EndComp
-$Comp
-L ATXMEGA32A4U IC1
-U 1 1 51159BBF
-P 5000 3950
-F 0 "IC1" H 3800 5580 50  0000 L BNN
-F 1 "ATXMEGA32A4U" H 6300 2350 50  0000 R BNN
-F 2 "TQFP44" H 3800 2400 50  0000 L CNN
-F 3 "http://www.atmel.com/Images/Atmel-8387-8-and16-bit-AVR-Microcontroller-XMEGA-A4U_Datasheet.pdf" H 5000 3950 60  0001 C CNN
-F 4 "ATXMEGA32A4U-AU-ND" H 5000 3950 60  0001 C CNN "Digi-Key Part Number"
-F 5 "ATXMEGA128A4U-AU-ND	" H 5000 3950 60  0001 C CNN "Alternative"
-	1    5000 3950
 	1    0    0    -1
 $EndComp
@@
 	10100 1300 10100 1950
 Connection ~ 9750 1300
+$Comp
+L ATXMEGA128A4U IC?
+U 1 1 52234FEA
+P 5000 3950
+F 0 "IC?" H 3800 5580 50  0000 L BNN
+F 1 "ATXMEGA128A4U" H 6300 2350 50  0000 R BNN
+F 2 "TQFP44" H 3800 2400 50  0000 L CNN
+F 3 "http://www.atmel.com/Images/Atmel-8387-8-and16-bit-AVR-Microcontroller-XMEGA-A4U_Datasheet.pdf" H 5000 3950 60  0001 C CNN
+F 4 "ATXMEGA128A4U-AU-ND" H 5000 3950 60  0001 C CNN "Digi-Key Part Number"
+F 5 "ATXMEGA128A4U-AU" H 5000 3950 60  0001 C CNN "Manufacturer Part Number"
+	1    5000 3950
+	1    0    0    -1
+$EndComp
 $EndSCHEMATC

Commit message: annotation
Signed-off-by: TheTesla <stefan.helmert@gmx.net>
Parts:
- gave numbers to parts that had none: 1
Changed lines of the file:
@@
-EESchema Schematic File Version 2  date 01.09.2013 16:25:21
+EESchema Schematic File Version 2  date 01.09.2013 19:38:16
 LIBS:atmel
 LIBS:libtest
@@
 Connection ~ 9750 1300
 $Comp
-L ATXMEGA128A4U IC?
+L ATXMEGA128A4U IC1
 U 1 1 52234FEA
 P 5000 3950
-F 0 "IC?" H 3800 5580 50  0000 L BNN
+F 0 "IC1" H 3800 5580 50  0000 L BNN
 F 1 "ATXMEGA128A4U" H 6300 2350 50  0000 R BNN
 F 2 "TQFP44" H 3800 2400 50  0000 L CNN

Commit message: better package for D4, D4 shifted down
Signed-off-by: TheTesla <stefan.helmert@gmx.net>
Parts:
- D3, D5: footprint SM0805 -> LED-0805
- D4: footprint SOT363 -> SOT-363
- P4: footprint ZX62-B-5PA -> MICRO-B_USB
