File: ATXMega128_USB_TEST_Board/ATXMega128_USB_TEST_Board.sch (KiCad schematic (older format))
At the start: 42 parts

Commit message: Test-Board schematic nearly ready
Signed-off-by: TheTesla <stefan.helmert@gmx.net>
Parts:
- added C? (x3): 10u, ~, symbol C
- added CON?: BARREL_JACK, symbol BARREL_JACK
- added D?: LED, ~, symbol LED
- added R? (x13): 10k, ~, symbol R
- added R? (x2): 100k, ~, symbol R
- added R?: 1k, ~, symbol R
Connections:
- wire segments 97 -> 171
Other:
- moved on the sheet: C?, D?, J?, Q?, R?

Commit message: ATXMega_Breaout-Footprint designed, Testboard PCB started
Signed-off-by: TheTesla <stefan.helmert@gmx.net>
Parts:
- removed IC?: ATXMEGA128A4U_BOARD, DIL40, symbol ATXMEGA128A4U_BOARD
- added D2, D3: LED, ~, symbol LED
- added IC?: ATXMEGA128A4U_BOARD, ATXMega128a4u_Breakout, symbol ATXMEGA128A4U_BOARD
- added R2, R6: 1k, ~, symbol R
- D1: renamed from D?; Notes (none) -> gelb
- D10, D11, D13, D14, D6, D7: renamed from D?; Notes (none) -> rot
- D12, D4: renamed from D?; Notes (none) -> gruen
- D5: renamed from D?; value DIODE -> 1N4148
- R12: renamed from R?; value R -> 1k
- R29, R30: renamed from R?; value 3k3 -> 10k
- gave numbers to parts that had none: 49
Connections:
- wire segments 171 -> 178
Other:
- moved on the sheet: D4, R12, R20, R24

Commit message: Testboard PCB designed
Signed-off-by: TheTesla <stefan.helmert@gmx.net>
Parts:
- gave numbers to parts that had none: 1
Connections:
- wire segments 178 -> 181
Other:
- moved on the sheet: D10, D13, R31, R37
Changed lines of the file:
@@
-EESchema Schematic File Version 2  date 10.09.2013 21:48:23
+EESchema Schematic File Version 2  date 11.09.2013 21:01:17
 LIBS:power
 LIBS:device
@@
 Sheet 1 1
 Title ""
-Date "10 sep 2013"
+Date "11 sep 2013"
 Rev ""
 Comp ""
@@
 $EndDescr
 $Comp
-L GND #PWR01
+L GND #PWR13
 U 1 1 522AF6D6
 P 5000 5750
-F 0 "#PWR01" H 5000 5750 30  0001 C CNN
+F 0 "#PWR13" H 5000 5750 30  0001 C CNN
 F 1 "GND" H 5000 5680 30  0001 C CNN
 F 2 "" H 5000 5750 60  0000 C CNN
@@
 $EndComp
 $Comp
-L +3,3V #PWR02
+L +3,3V #PWR11
 U 1 1 522AF769
 P 4300 1900
-F 0 "#PWR02" H 4300 1860 30  0001 C CNN
+F 0 "#PWR11" H 4300 1860 30  0001 C CNN
 F 1 "+3,3V" H 4300 2010 30  0000 C CNN
 F 2 "" H 4300 1900 60  0000 C CNN
@@
 $EndComp
 $Comp
-L GND #PWR03
+L GND #PWR17
 U 1 1 522B010E
 P 8400 3850
-F 0 "#PWR03" H 8400 3850 30  0001 C CNN
+F 0 "#PWR17" H 8400 3850 30  0001 C CNN
 F 1 "GND" H 8400 3780 30  0001 C CNN
 F 2 "" H 8400 3850 60  0000 C CNN
@@
 L LED D10
 U 1 1 522B1ED4
-P 9300 3300
-F 0 "D10" H 9300 3400 50  0000 C CNN
-F 1 "LED" H 9300 3200 50  0000 C CNN
-F 2 "~" H 9300 3300 60  0000 C CNN
-F 3 "~" H 9300 3300 60  0000 C CNN
-F 4 "rot" H 9300 3300 60  0001 C CNN "Notes"
-	1    9300 3300
+P 9300 2700
+F 0 "D10" H 9300 2800 50  0000 C CNN
+F 1 "LED" H 9300 2600 50  0000 C CNN
+F 2 "~" H 9300 2700 60  0000 C CNN
+F 3 "~" H 9300 2700 60  0000 C CNN
+F 4 "rot" H 9300 2700 60  0001 C CNN "Notes"
+	1    9300 2700
 	0    1    1    0
 $EndComp
@@
 L R R31
 U 1 1 522B1EEB
-P 9300 2750
-F 0 "R31" V 9380 2750 40  0000 C CNN
-F 1 "1k" V 9307 2751 40  0000 C CNN
-F 2 "~" V 9230 2750 30  0000 C CNN
-F 3 "~" H 9300 2750 30  0000 C CNN
-	1    9300 2750
-	1    0    0    -1
-$EndComp
-$Comp
-L +3,3V #PWR04
+P 9300 3250
+F 0 "R31" V 9380 3250 40  0000 C CNN
+F 1 "1k" V 9307 3251 40  0000 C CNN
+F 2 "~" V 9230 3250 30  0000 C CNN
+F 3 "~" H 9300 3250 30  0000 C CNN
+	1    9300 3250
+	1    0    0    -1
+$EndComp
+$Comp
+L +3,3V #PWR18
 U 1 1 522B1EF8
 P 9300 2350
-F 0 "#PWR04" H 9300 2310 30  0001 C CNN
+F 0 "#PWR18" H 9300 2310 30  0001 C CNN
 F 1 "+3,3V" H 9300 2460 30  0000 C CNN
 F 2 "" H 9300 2350 60  0000 C CNN
@@
 $EndComp
 $Comp
-L PWR_FLAG #FLG05
+L PWR_FLAG #FLG1
 U 1 1 522B20FF
 P 4500 1950
-F 0 "#FLG05" H 4500 2045 30  0001 C CNN
+F 0 "#FLG1" H 4500 2045 30  0001 C CNN
 F 1 "PWR_FLAG" H 4500 2130 30  0000 C CNN
 F 2 "" H 4500 1950 60  0000 C CNN
@@
 $EndComp
 $Comp
-L PWR_FLAG #FLG06
+L PWR_FLAG #FLG2
 U 1 1 522B21CD
 P 8350 700
-F 0 "#FLG06" H 8350 795 30  0001 C CNN
+F 0 "#FLG2" H 8350 795 30  0001 C CNN
 F 1 "PWR_FLAG" H 8350 880 30  0000 C CNN
 F 2 "" H 8350 700 60  0000 C CNN
@@
 $EndComp
 $Comp
-L GND #PWR07
+L GND #PWR19
 U 1 1 522B27F2
 P 9300 6100
-F 0 "#PWR07" H 9300 6100 30  0001 C CNN
+F 0 "#PWR19" H 9300 6100 30  0001 C CNN
 F 1 "GND" H 9300 6030 30  0001 C CNN
 F 2 "" H 9300 6100 60  0000 C CNN
@@
 $EndComp
 $Comp
-L +3,3V #PWR08
+L +3,3V #PWR15
 U 1 1 522B2AC7
 P 6600 5600
-F 0 "#PWR08" H 6600 5560 30  0001 C CNN
+F 0 "#PWR15" H 6600 5560 30  0001 C CNN
 F 1 "+3,3V" H 6600 5710 30  0000 C CNN
 F 2 "" H 6600 5600 60  0000 C CNN
@@
 $EndComp
 $Comp
-L GND #PWR09
+L GND #PWR20
 U 1 1 522C252A
 P 9700 3850
-F 0 "#PWR09" H 9700 3850 30  0001 C CNN
+F 0 "#PWR20" H 9700 3850 30  0001 C CNN
 F 1 "GND" H 9700 3780 30  0001 C CNN
 F 2 "" H 9700 3850 60  0000 C CNN
@@
 L LED D13
 U 1 1 522C2531
-P 10750 3300
-F 0 "D13" H 10750 3400 50  0000 C CNN
-F 1 "LED" H 10750 3200 50  0000 C CNN
-F 2 "~" H 10750 3300 60  0000 C CNN
-F 3 "~" H 10750 3300 60  0000 C CNN
-F 4 "rot" H 10750 3300 60  0001 C CNN "Notes"
-	1    10750 3300
+P 10750 2700
+F 0 "D13" H 10750 2800 50  0000 C CNN
+F 1 "LED" H 10750 2600 50  0000 C CNN
+F 2 "~" H 10750 2700 60  0000 C CNN
+F 3 "~" H 10750 2700 60  0000 C CNN
+F 4 "rot" H 10750 2700 60  0001 C CNN "Notes"
+	1    10750 2700
 	0    1    1    0
 $EndComp
@@
 L R R37
 U 1 1 522C2537
-P 10750 2750
-F 0 "R37" V 10830 2750 40  0000 C CNN
-F 1 "1k" V 10757 2751 40  0000 C CNN
-F 2 "~" V 10680 2750 30  0000 C CNN
-F 3 "~" H 10750 2750 30  0000 C CNN
-	1    10750 2750
-	1    0    0    -1
-$EndComp
-$Comp
-L +3,3V #PWR010
+P 10750 3250
+F 0 "R37" V 10830 3250 40  0000 C CNN
+F 1 "1k" V 10757 3251 40  0000 C CNN
+F 2 "~" V 10680 3250 30  0000 C CNN
+F 3 "~" H 10750 3250 30  0000 C CNN
+	1    10750 3250
+	1    0    0    -1
+$EndComp
+$Comp
+L +3,3V #PWR21
 U 1 1 522C253D
 P 10750 2350
-F 0 "#PWR010" H 10750 2310 30  0001 C CNN
+F 0 "#PWR21" H 10750 2310 30  0001 C CNN
 F 1 "+3,3V" H 10750 2460 30  0000 C CNN
 F 2 "" H 10750 2350 60  0000 C CNN
@@
 $EndComp
 $Comp
-L GND #PWR011
+L GND #PWR22
 U 1 1 522C2587
 P 10750 6100
-F 0 "#PWR011" H 10750 6100 30  0001 C CNN
+F 0 "#PWR22" H 10750 6100 30  0001 C CNN
 F 1 "GND" H 10750 6030 30  0001 C CNN
 F 2 "" H 10750 6100 60  0000 C CNN
@@
 $EndComp
 $Comp
-L GND #PWR012
+L GND #PWR14
 U 1 1 522C274B
 P 6500 1850
-F 0 "#PWR012" H 6500 1850 30  0001 C CNN
+F 0 "#PWR14" H 6500 1850 30  0001 C CNN
 F 1 "GND" H 6500 1780 30  0001 C CNN
 F 2 "" H 6500 1850 60  0000 C CNN
@@
 $EndComp
 $Comp
-L +3,3V #PWR013
+L +3,3V #PWR10
 U 1 1 522C76BF
 P 3400 1150
-F 0 "#PWR013" H 3400 1110 30  0001 C CNN
+F 0 "#PWR10" H 3400 1110 30  0001 C CNN
 F 1 "+3,3V" H 3400 1260 30  0000 C CNN
 F 2 "" H 3400 1150 60  0000 C CNN
@@
 $EndComp
 $Comp
-L GND #PWR014
+L GND #PWR8
 U 1 1 522C77CC
 P 2900 1800
-F 0 "#PWR014" H 2900 1800 30  0001 C CNN
+F 0 "#PWR8" H 2900 1800 30  0001 C CNN
 F 1 "GND" H 2900 1730 30  0001 C CNN
 F 2 "" H 2900 1800 60  0000 C CNN
@@
 $EndComp
 $Comp
-L GND #PWR015
+L GND #PWR3
 U 1 1 522C7FEA
 P 1850 1800
-F 0 "#PWR015" H 1850 1800 30  0001 C CNN
+F 0 "#PWR3" H 1850 1800 30  0001 C CNN
 F 1 "GND" H 1850 1730 30  0001 C CNN
 F 2 "" H 1850 1800 60  0000 C CNN
@@
 $EndComp
 $Comp
-L +8V #PWR016
+L +8V #PWR7
 U 1 1 522C810D
 P 2350 1100
-F 0 "#PWR016" H 2350 1070 20  0001 C CNN
+F 0 "#PWR7" H 2350 1070 20  0001 C CNN
 F 1 "+8V" H 2350 1210 30  0000 C CNN
 F 2 "" H 2350 1100 60  0000 C CNN
@@
 $EndComp
 $Comp
-L +8V #PWR017
+L +8V #PWR16
 U 1 1 522C8243
 P 8100 650
-F 0 "#PWR017" H 8100 620 20  0001 C CNN
+F 0 "#PWR16" H 8100 620 20  0001 C CNN
 F 1 "+8V" H 8100 760 30  0000 C CNN
 F 2 "" H 8100 650 60  0000 C CNN
@@
 $EndComp
 $Comp
-L +3,3V #PWR018
+L +3,3V #PWR12
 U 1 1 522CCEFB
 P 4950 1600
-F 0 "#PWR018" H 4950 1560 30  0001 C CNN
+F 0 "#PWR12" H 4950 1560 30  0001 C CNN
 F 1 "+3,3V" H 4950 1710 30  0000 C CNN
 F 2 "" H 4950 1600 60  0000 C CNN
@@
 $EndComp
 $Comp
-L GND #PWR019
+L GND #PWR6
 U 1 1 522CE393
 P 2300 2600
-F 0 "#PWR019" H 2300 2600 30  0001 C CNN
+F 0 "#PWR6" H 2300 2600 30  0001 C CNN
 F 1 "GND" H 2300 2530 30  0001 C CNN
 F 2 "" H 2300 2600 60  0000 C CNN
@@
 $EndComp
 $Comp
-L +3,3V #PWR020
+L +3,3V #PWR4
 U 1 1 522CE3FC
 P 2100 2650
-F 0 "#PWR020" H 2100 2610 30  0001 C CNN
+F 0 "#PWR4" H 2100 2610 30  0001 C CNN
 F 1 "+3,3V" H 2100 2760 30  0000 C CNN
 F 2 "" H 2100 2650 60  0000 C CNN
@@
 	9300 2350 9300 2500
 Wire Wire Line
-	9300 3000 9300 3100
+	9300 2900 9300 3000
 Wire Wire Line
 	9300 3500 9300 3650
@@
 	10750 2350 10750 2500
 Wire Wire Line
-	10750 3000 10750 3100
+	10750 2900 10750 3000
 Wire Wire Line
 	10750 3500 10750 3650
@@
 	7100 4650 7000 4650
 Wire Wire Line
-	7000 4650 7000 4750
-Wire Wire Line
-	7000 4750 6600 4750
-Wire Wire Line
-	7250 4650 7250 4550
-Wire Wire Line
-	7250 4550 6600 4550
+	7000 4650 7000 4850
+Wire Wire Line
+	7250 4450 7250 4650
 Wire Wire Line
 	6450 5000 6450 4900
-Wire Wire Line
-	6450 4900 6600 4900
-Wire Wire Line
-	6600 4900 6600 4850
-Wire Wire Line
-	6950 5000 6950 4650
-Wire Wire Line
-	6950 4650 6600 4650
 Wire Wire Line
 	6600 4050 6700 4050
@@
 $EndComp
 $Comp
-L +3,3V #PWR021
+L +3,3V #PWR1
 U 1 1 522E60D1
 P 1400 2600
-F 0 "#PWR021" H 1400 2560 30  0001 C CNN
+F 0 "#PWR1" H 1400 2560 30  0001 C CNN
 F 1 "+3,3V" H 1400 2710 30  0000 C CNN
 F 2 "" H 1400 2600 60  0000 C CNN
@@
 	1400 3750 1400 3900
 $Comp
-L GND #PWR022
+L GND #PWR2
 U 1 1 522E60DA
 P 1400 3900
-F 0 "#PWR022" H 1400 3900 30  0001 C CNN
+F 0 "#PWR2" H 1400 3900 30  0001 C CNN
 F 1 "GND" H 1400 3830 30  0001 C CNN
 F 2 "" H 1400 3900 60  0000 C CNN
@@
 	2950 6450 2950 6600
 $Comp
-L GND #PWR023
+L GND #PWR9
 U 1 1 522F63C1
 P 2950 6600
-F 0 "#PWR023" H 2950 6600 30  0001 C CNN
+F 0 "#PWR9" H 2950 6600 30  0001 C CNN
 F 1 "GND" H 2950 6530 30  0001 C CNN
 F 2 "" H 2950 6600 60  0000 C CNN
@@
 	2150 6450 2150 6600
 $Comp
-L GND #PWR024
+L GND #PWR5
 U 1 1 522F65BC
 P 2150 6600
-F 0 "#PWR024" H 2150 6600 30  0001 C CNN
+F 0 "#PWR5" H 2150 6600 30  0001 C CNN
 F 1 "GND" H 2150 6530 30  0001 C CNN
 F 2 "" H 2150 6600 60  0000 C CNN
@@
 Connection ~ 1300 1700
 $Comp
-L ATXMEGA128A4U_BOARD IC?
+L ATXMEGA128A4U_BOARD IC1
 U 1 1 522F79D7
 P 5100 3850
-F 0 "IC?" H 3900 5480 50  0000 L BNN
+F 0 "IC1" H 3900 5480 50  0000 L BNN
 F 1 "ATXMEGA128A4U_BOARD" H 6400 2250 50  0000 R BNN
 F 2 "ATXMega128a4u_Breakout" H 3900 2300 50  0000 L CNN
@@
 	1    0    0    -1
 $EndComp
+Wire Wire Line
+	6450 4900 6800 4900
+Wire Wire Line
+	6800 4900 6800 4750
+Wire Wire Line
+	6800 4750 6600 4750
+Wire Wire Line
+	6950 5000 6950 4550
+Wire Wire Line
+	6950 4550 6600 4550
+Wire Wire Line
+	7000 4850 6600 4850
+Wire Wire Line
+	6600 4650 6850 4650
+Wire Wire Line
+	6850 4650 6850 4450
+Wire Wire Line
+	6850 4450 7250 4450
 $EndSCHEMATC

Commit message: Power Supply Diode added, Board Edge Cuts added
Signed-off-by: TheTesla <stefan.helmert@gmx.net>
Parts:
- added D?: 1N4148, ~, symbol DIODE
Connections:
- wire segments 181 -> 186
Changed lines of the file:
@@
-EESchema Schematic File Version 2  date 11.09.2013 21:01:17
+EESchema Schematic File Version 2  date 13.09.2013 22:25:03
 LIBS:power
 LIBS:device
@@
 Sheet 1 1
 Title ""
-Date "11 sep 2013"
+Date "13 sep 2013"
 Rev ""
 Comp ""
@@
 $EndDescr
 $Comp
-L GND #PWR13
+L GND #PWR01
 U 1 1 522AF6D6
 P 5000 5750
-F 0 "#PWR13" H 5000 5750 30  0001 C CNN
+F 0 "#PWR01" H 5000 5750 30  0001 C CNN
 F 1 "GND" H 5000 5680 30  0001 C CNN
 F 2 "" H 5000 5750 60  0000 C CNN
@@
 $EndComp
 $Comp
-L +3,3V #PWR11
+L +3,3V #PWR02
 U 1 1 522AF769
 P 4300 1900
-F 0 "#PWR11" H 4300 1860 30  0001 C CNN
+F 0 "#PWR02" H 4300 1860 30  0001 C CNN
 F 1 "+3,3V" H 4300 2010 30  0000 C CNN
 F 2 "" H 4300 1900 60  0000 C CNN
@@
 $EndComp
 $Comp
-L GND #PWR17
+L GND #PWR03
 U 1 1 522B010E
 P 8400 3850
-F 0 "#PWR17" H 8400 3850 30  0001 C CNN
+F 0 "#PWR03" H 8400 3850 30  0001 C CNN
 F 1 "GND" H 8400 3780 30  0001 C CNN
 F 2 "" H 8400 3850 60  0000 C CNN
@@
 $EndComp
 $Comp
-L +3,3V #PWR18
+L +3,3V #PWR04
 U 1 1 522B1EF8
 P 9300 2350
-F 0 "#PWR18" H 9300 2310 30  0001 C CNN
+F 0 "#PWR04" H 9300 2310 30  0001 C CNN
 F 1 "+3,3V" H 9300 2460 30  0000 C CNN
 F 2 "" H 9300 2350 60  0000 C CNN
@@
 $EndComp
 $Comp
-L PWR_FLAG #FLG1
+L PWR_FLAG #FLG05
 U 1 1 522B20FF
 P 4500 1950
-F 0 "#FLG1" H 4500 2045 30  0001 C CNN
+F 0 "#FLG05" H 4500 2045 30  0001 C CNN
 F 1 "PWR_FLAG" H 4500 2130 30  0000 C CNN
 F 2 "" H 4500 1950 60  0000 C CNN
@@
 $EndComp
 $Comp
-L PWR_FLAG #FLG2
+L PWR_FLAG #FLG06
 U 1 1 522B21CD
 P 8350 700
-F 0 "#FLG2" H 8350 795 30  0001 C CNN
+F 0 "#FLG06" H 8350 795 30  0001 C CNN
 F 1 "PWR_FLAG" H 8350 880 30  0000 C CNN
 F 2 "" H 8350 700 60  0000 C CNN
@@
 $EndComp
 $Comp
-L GND #PWR19
+L GND #PWR07
 U 1 1 522B27F2
 P 9300 6100
-F 0 "#PWR19" H 9300 6100 30  0001 C CNN
+F 0 "#PWR07" H 9300 6100 30  0001 C CNN
 F 1 "GND" H 9300 6030 30  0001 C CNN
 F 2 "" H 9300 6100 60  0000 C CNN
@@
 $EndComp
 $Comp
-L +3,3V #PWR15
+L +3,3V #PWR08
 U 1 1 522B2AC7
 P 6600 5600
-F 0 "#PWR15" H 6600 5560 30  0001 C CNN
+F 0 "#PWR08" H 6600 5560 30  0001 C CNN
 F 1 "+3,3V" H 6600 5710 30  0000 C CNN
 F 2 "" H 6600 5600 60  0000 C CNN
@@
 $EndComp
 $Comp
-L GND #PWR20
+L GND #PWR09
 U 1 1 522C252A
 P 9700 3850
-F 0 "#PWR20" H 9700 3850 30  0001 C CNN
+F 0 "#PWR09" H 9700 3850 30  0001 C CNN
 F 1 "GND" H 9700 3780 30  0001 C CNN
 F 2 "" H 9700 3850 60  0000 C CNN
@@
 $EndComp
 $Comp
-L +3,3V #PWR21
+L +3,3V #PWR010
 U 1 1 522C253D
 P 10750 2350
-F 0 "#PWR21" H 10750 2310 30  0001 C CNN
+F 0 "#PWR010" H 10750 2310 30  0001 C CNN
 F 1 "+3,3V" H 10750 2460 30  0000 C CNN
 F 2 "" H 10750 2350 60  0000 C CNN
@@
 $EndComp
 $Comp
-L GND #PWR22
+L GND #PWR011
 U 1 1 522C2587
 P 10750 6100
-F 0 "#PWR22" H 10750 6100 30  0001 C CNN
+F 0 "#PWR011" H 10750 6100 30  0001 C CNN
 F 1 "GND" H 10750 6030 30  0001 C CNN
 F 2 "" H 10750 6100 60  0000 C CNN
@@
 $EndComp
 $Comp
-L GND #PWR14
+L GND #PWR012
 U 1 1 522C274B
 P 6500 1850
-F 0 "#PWR14" H 6500 1850 30  0001 C CNN
+F 0 "#PWR012" H 6500 1850 30  0001 C CNN
 F 1 "GND" H 6500 1780 30  0001 C CNN
 F 2 "" H 6500 1850 60  0000 C CNN
@@
 $EndComp
 $Comp
-L +3,3V #PWR10
+L +3,3V #PWR013
 U 1 1 522C76BF
 P 3400 1150
-F 0 "#PWR10" H 3400 1110 30  0001 C CNN
+F 0 "#PWR013" H 3400 1110 30  0001 C CNN
 F 1 "+3,3V" H 3400 1260 30  0000 C CNN
 F 2 "" H 3400 1150 60  0000 C CNN
@@
 $EndComp
 $Comp
-L GND #PWR8
+L GND #PWR014
 U 1 1 522C77CC
 P 2900 1800
-F 0 "#PWR8" H 2900 1800 30  0001 C CNN
+F 0 "#PWR014" H 2900 1800 30  0001 C CNN
 F 1 "GND" H 2900 1730 30  0001 C CNN
 F 2 "" H 2900 1800 60  0000 C CNN
@@
 $EndComp
 $Comp
-L GND #PWR3
+L GND #PWR015
 U 1 1 522C7FEA
 P 1850 1800
-F 0 "#PWR3" H 1850 1800 30  0001 C CNN
+F 0 "#PWR015" H 1850 1800 30  0001 C CNN
 F 1 "GND" H 1850 1730 30  0001 C CNN
 F 2 "" H 1850 1800 60  0000 C CNN
@@
 $EndComp
 $Comp
-L +8V #PWR7
+L +8V #PWR016
 U 1 1 522C810D
 P 2350 1100
-F 0 "#PWR7" H 2350 1070 20  0001 C CNN
+F 0 "#PWR016" H 2350 1070 20  0001 C CNN
 F 1 "+8V" H 2350 1210 30  0000 C CNN
 F 2 "" H 2350 1100 60  0000 C CNN
@@
 $EndComp
 $Comp
-L +8V #PWR16
+L +8V #PWR017
 U 1 1 522C8243
 P 8100 650
-F 0 "#PWR16" H 8100 620 20  0001 C CNN
+F 0 "#PWR017" H 8100 620 20  0001 C CNN
 F 1 "+8V" H 8100 760 30  0000 C CNN
 F 2 "" H 8100 650 60  0000 C CNN
@@
 $EndComp
 $Comp
-L +3,3V #PWR12
+L +3,3V #PWR018
 U 1 1 522CCEFB
 P 4950 1600
-F 0 "#PWR12" H 4950 1560 30  0001 C CNN
+F 0 "#PWR018" H 4950 1560 30  0001 C CNN
 F 1 "+3,3V" H 4950 1710 30  0000 C CNN
 F 2 "" H 4950 1600 60  0000 C CNN
@@
 $EndComp
 $Comp
-L GND #PWR6
+L GND #PWR019
 U 1 1 522CE393
 P 2300 2600
-F 0 "#PWR6" H 2300 2600 30  0001 C CNN
+F 0 "#PWR019" H 2300 2600 30  0001 C CNN
 F 1 "GND" H 2300 2530 30  0001 C CNN
 F 2 "" H 2300 2600 60  0000 C CNN
@@
 $EndComp
 $Comp
-L +3,3V #PWR4
+L +3,3V #PWR020
 U 1 1 522CE3FC
 P 2100 2650
-F 0 "#PWR4" H 2100 2610 30  0001 C CNN
+F 0 "#PWR020" H 2100 2610 30  0001 C CNN
 F 1 "+3,3V" H 2100 2760 30  0000 C CNN
 F 2 "" H 2100 2650 60  0000 C CNN
@@
 	3350 1700 3350 1650
 Wire Wire Line
-	1400 1250 1400 1200
-Wire Wire Line
-	1200 1200 1450 1200
+	1400 900  1400 1250
 Wire Wire Line
 	1400 1650 1400 1700
@@
 $EndComp
 Connection ~ 1400 1700
-Wire Wire Line
-	1200 1500 1200 1200
 Connection ~ 1400 1200
 $Comp
@@
 $EndComp
 $Comp
-L +3,3V #PWR1
+L +3,3V #PWR021
 U 1 1 522E60D1
 P 1400 2600
-F 0 "#PWR1" H 1400 2560 30  0001 C CNN
+F 0 "#PWR021" H 1400 2560 30  0001 C CNN
 F 1 "+3,3V" H 1400 2710 30  0000 C CNN
 F 2 "" H 1400 2600 60  0000 C CNN
@@
 	1400 3750 1400 3900
 $Comp
-L GND #PWR2
+L GND #PWR022
 U 1 1 522E60DA
 P 1400 3900
-F 0 "#PWR2" H 1400 3900 30  0001 C CNN
+F 0 "#PWR022" H 1400 3900 30  0001 C CNN
 F 1 "GND" H 1400 3830 30  0001 C CNN
 F 2 "" H 1400 3900 60  0000 C CNN
@@
 	2950 6450 2950 6600
 $Comp
-L GND #PWR9
+L GND #PWR023
 U 1 1 522F63C1
 P 2950 6600
-F 0 "#PWR9" H 2950 6600 30  0001 C CNN
+F 0 "#PWR023" H 2950 6600 30  0001 C CNN
 F 1 "GND" H 2950 6530 30  0001 C CNN
 F 2 "" H 2950 6600 60  0000 C CNN
@@
 	2150 6450 2150 6600
 $Comp
-L GND #PWR5
+L GND #PWR024
 U 1 1 522F65BC
 P 2150 6600
-F 0 "#PWR5" H 2150 6600 30  0001 C CNN
+F 0 "#PWR024" H 2150 6600 30  0001 C CNN
 F 1 "GND" H 2150 6530 30  0001 C CNN
 F 2 "" H 2150 6600 60  0000 C CNN
@@
 Wire Wire Line
 	6850 4450 7250 4450
+$Comp
+L DIODE D?
+U 1 1 52337484
+P 1150 900
+F 0 "D?" H 1150 1000 40  0000 C CNN
+F 1 "1N4148" H 1150 800 40  0000 C CNN
+F 2 "~" H 1150 900 60  0000 C CNN
+F 3 "~" H 1150 900 60  0000 C CNN
+	1    1150 900
+	1    0    0    -1
+$EndComp
+Wire Wire Line
+	1350 900  1400 900
+Wire Wire Line
+	1400 1200 1450 1200
+Wire Wire Line
+	1200 1500 1250 1500
+Wire Wire Line
+	1250 1500 1250 1250
+Wire Wire Line
+	1250 1250 850  1250
+Wire Wire Line
+	850  1250 850  900
+Wire Wire Line
+	850  900  950  900
 $EndSCHEMATC

Commit message: Testboard complete
Signed-off-by: TheTesla <stefan.helmert@gmx.net>
Parts:
- removed U1: MC78L08ACH, SOT-89, symbol MC78L08ACH
- added C5: 100n, ~, symbol C
- added C6: 100u, ~, symbol CP1
- added C7, C8: 10u, ~, symbol CP1
- added D16, D17: 4V7, ~, symbol ZENER
- added U1: MC78L12ACH, SOT-89, symbol MC78L12ACH
- C1, C2: value 10u -> 330n
- C3: value 10u -> 100n
- D8: value 6V2 -> 5V6
- D9: value 6V2 -> 9V6
- R20: value 1k -> 10k
- R24: value 220 -> 470
- gave numbers to parts that had none: 1
Connections:
- net labels added: +12V
- net labels removed: +8V
- wire segments 186 -> 199
Other:
- moved on the sheet: C1, C2, C3, R20, R24, R28, U2

Commit message: Testboard updated, Testsoftware ready
Signed-off-by: TheTesla <stefan.helmert@gmx.net>
Parts:
- R1, R10, R12, R13, R2, R25, R26, R27, R28, R31, R32, R34, R35, R36, R37, R38, R6: value 1k -> 820
- R19, R21: value 100k -> 200k
- R7, R9: value 10k -> 200k
Changed lines of the file:
@@
-EESchema Schematic File Version 2  date 15.09.2013 13:13:35
+EESchema Schematic File Version 2  date 10.10.2013 19:16:10
 LIBS:power
 LIBS:device
@@
 Sheet 1 1
 Title ""
-Date "14 sep 2013"
+Date "10 oct 2013"
 Rev ""
 Comp ""
@@
 P 9300 3250
 F 0 "R31" V 9380 3250 40  0000 C CNN
-F 1 "1k" V 9307 3251 40  0000 C CNN
+F 1 "820" V 9307 3251 40  0000 C CNN
 F 2 "~" V 9230 3250 30  0000 C CNN
 F 3 "~" H 9300 3250 30  0000 C CNN
@@
 P 9800 4150
 F 0 "R34" V 9880 4150 40  0000 C CNN
-F 1 "1k" V 9807 4151 40  0000 C CNN
+F 1 "820" V 9807 4151 40  0000 C CNN
 F 2 "~" V 9730 4150 30  0000 C CNN
 F 3 "~" H 9800 4150 30  0000 C CNN
@@
 P 9300 5200
 F 0 "R32" V 9380 5200 40  0000 C CNN
-F 1 "1k" V 9307 5201 40  0000 C CNN
+F 1 "820" V 9307 5201 40  0000 C CNN
 F 2 "~" V 9230 5200 30  0000 C CNN
 F 3 "~" H 9300 5200 30  0000 C CNN
@@
 P 6050 5600
 F 0 "R12" V 6130 5600 40  0000 C CNN
-F 1 "1k" V 6057 5601 40  0000 C CNN
+F 1 "820" V 6057 5601 40  0000 C CNN
 F 2 "~" V 5980 5600 30  0000 C CNN
 F 3 "~" H 6050 5600 30  0000 C CNN
@@
 P 8700 3850
 F 0 "R27" V 8780 3850 40  0000 C CNN
-F 1 "1k" V 8707 3851 40  0000 C CNN
+F 1 "820" V 8707 3851 40  0000 C CNN
 F 2 "~" V 8630 3850 30  0000 C CNN
 F 3 "~" H 8700 3850 30  0000 C CNN
@@
 P 8600 4600
 F 0 "R28" V 8680 4600 40  0000 C CNN
-F 1 "1k" V 8607 4601 40  0000 C CNN
+F 1 "820" V 8607 4601 40  0000 C CNN
 F 2 "~" V 8530 4600 30  0000 C CNN
 F 3 "~" H 8600 4600 30  0000 C CNN
@@
 P 10750 3250
 F 0 "R37" V 10830 3250 40  0000 C CNN
-F 1 "1k" V 10757 3251 40  0000 C CNN
+F 1 "820" V 10757 3251 40  0000 C CNN
 F 2 "~" V 10680 3250 30  0000 C CNN
 F 3 "~" H 10750 3250 30  0000 C CNN
@@
 P 10050 3850
 F 0 "R35" V 10130 3850 40  0000 C CNN
-F 1 "1k" V 10057 3851 40  0000 C CNN
+F 1 "820" V 10057 3851 40  0000 C CNN
 F 2 "~" V 9980 3850 30  0000 C CNN
 F 3 "~" H 10050 3850 30  0000 C CNN
@@
 P 10750 5200
 F 0 "R38" V 10830 5200 40  0000 C CNN
-F 1 "1k" V 10757 5201 40  0000 C CNN
+F 1 "820" V 10757 5201 40  0000 C CNN
 F 2 "~" V 10680 5200 30  0000 C CNN
 F 3 "~" H 10750 5200 30  0000 C CNN
@@
 P 10050 4600
 F 0 "R36" V 10130 4600 40  0000 C CNN
-F 1 "1k" V 10057 4601 40  0000 C CNN
+F 1 "820" V 10057 4601 40  0000 C CNN
 F 2 "~" V 9980 4600 30  0000 C CNN
 F 3 "~" H 10050 4600 30  0000 C CNN
@@
 P 6050 1300
 F 0 "R13" V 6130 1300 40  0000 C CNN
-F 1 "1k" V 6057 1301 40  0000 C CNN
+F 1 "820" V 6057 1301 40  0000 C CNN
 F 2 "~" V 5980 1300 30  0000 C CNN
 F 3 "~" H 6050 1300 30  0000 C CNN
@@
 P 8650 1550
 F 0 "R26" V 8730 1550 40  0000 C CNN
-F 1 "1k" V 8657 1551 40  0000 C CNN
+F 1 "820" V 8657 1551 40  0000 C CNN
 F 2 "~" V 8580 1550 30  0000 C CNN
 F 3 "~" H 8650 1550 30  0000 C CNN
@@
 P 8500 1550
 F 0 "R25" V 8580 1550 40  0000 C CNN
-F 1 "1k" V 8507 1551 40  0000 C CNN
+F 1 "820" V 8507 1551 40  0000 C CNN
 F 2 "~" V 8430 1550 30  0000 C CNN
 F 3 "~" H 8500 1550 30  0000 C CNN
@@
 P 4950 1250
 F 0 "R10" V 5030 1250 40  0000 C CNN
-F 1 "1k" V 4957 1251 40  0000 C CNN
+F 1 "820" V 4957 1251 40  0000 C CNN
 F 2 "~" V 4880 1250 30  0000 C CNN
 F 3 "~" H 4950 1250 30  0000 C CNN
@@
 P 3300 3650
 F 0 "R7" V 3380 3650 40  0000 C CNN
-F 1 "10k" V 3307 3651 40  0000 C CNN
+F 1 "200k" V 3307 3651 40  0000 C CNN
 F 2 "~" V 3230 3650 30  0000 C CNN
 F 3 "~" H 3300 3650 30  0000 C CNN
@@
 P 3300 4850
 F 0 "R9" V 3380 4850 40  0000 C CNN
-F 1 "10k" V 3307 4851 40  0000 C CNN
+F 1 "200k" V 3307 4851 40  0000 C CNN
 F 2 "~" V 3230 4850 30  0000 C CNN
 F 3 "~" H 3300 4850 30  0000 C CNN
@@
 P 7250 4900
 F 0 "R21" V 7330 4900 40  0000 C CNN
-F 1 "100k" V 7257 4901 40  0000 C CNN
+F 1 "200k" V 7257 4901 40  0000 C CNN
 F 2 "~" V 7180 4900 30  0000 C CNN
 F 3 "~" H 7250 4900 30  0000 C CNN
@@
 P 7100 4900
 F 0 "R19" V 7180 4900 40  0000 C CNN
-F 1 "100k" V 7107 4901 40  0000 C CNN
+F 1 "200k" V 7107 4901 40  0000 C CNN
 F 2 "~" V 7030 4900 30  0000 C CNN
 F 3 "~" H 7100 4900 30  0000 C CNN
@@
 P 1400 3000
 F 0 "R1" V 1480 3000 40  0000 C CNN
-F 1 "1k" V 1407 3001 40  0000 C CNN
+F 1 "820" V 1407 3001 40  0000 C CNN
 F 2 "~" V 1330 3000 30  0000 C CNN
 F 3 "~" H 1400 3000 30  0000 C CNN
@@
 P 2950 5700
 F 0 "R6" V 3030 5700 40  0000 C CNN
-F 1 "1k" V 2957 5701 40  0000 C CNN
+F 1 "820" V 2957 5701 40  0000 C CNN
 F 2 "~" V 2880 5700 30  0000 C CNN
 F 3 "~" H 2950 5700 30  0000 C CNN
@@
 P 2150 5700
 F 0 "R2" V 2230 5700 40  0000 C CNN
-F 1 "1k" V 2157 5701 40  0000 C CNN
+F 1 "820" V 2157 5701 40  0000 C CNN
 F 2 "~" V 2080 5700 30  0000 C CNN
 F 3 "~" H 2150 5700 30  0000 C CNN
